Commit message: Initial commit

File: feeding_robot/description/feeding_robot_core.xacro (robot description, xacro)
@@ -4,20 +4,31 @@
   <!-- Adaptive Feeding Robot - 4 DOF Open Manipulator               -->
   <!-- Based on: Sadeghi Esfahlani et al. (2025)                    -->
+  <!-- CAD source: Auto Feeder SSE v222.step                        -->
   <!-- Joints: Base Y, Lower Z, Upper Z, Feeder                     -->
   <!-- Actuators: 4x Dynamixel XM430-W350R                          -->
   <!-- ============================================================ -->
   <!-- ==================== PARAMETERS ==================== -->
-  <!-- Dimensions (metres) - from paper Figure 2 -->
-  <xacro:property name="base_height" value="0.070"/>
+  <!-- Dimensions (metres) - measured from CAD bounding boxes -->
+  <!-- CAD assembly: X: -75 to 343mm, Y: -55 to 56mm, Z: -25 to 425mm -->
+  <!-- Base center at approximately X=-25, Y=0, Z=0 in CAD coords -->
+  <xacro:property name="base_height" value="0.088"/>
   <xacro:property name="base_radius" value="0.060"/>
   <xacro:property name="turntable_height" value="0.050"/>
   <xacro:property name="turntable_radius" value="0.045"/>
-  <!-- Shoulder height from base top to lower_z_joint axis -->
-  <xacro:property name="shoulder_height" value="0.16370"/>
-  <xacro:property name="lower_arm_length" value="0.20789"/>
+  <!-- Shoulder height: from base top to lower_z_joint axis -->
+  <!-- CAD: first motor (solid_000) center at Z=111.7mm, base top ~88mm -->
+  <!-- Joint axis at approximately Z=134mm from ground -->
+  <xacro:property name="shoulder_height" value="0.134"/>
+  <!-- Lower arm: vertical segment from shoulder to elbow -->
+  <!-- CAD: shoulder at Z~134mm, top of vertical arm at Z~338mm = 204mm -->
+  <xacro:property name="lower_arm_length" value="0.204"/>
   <xacro:property name="lower_arm_radius" value="0.025"/>
-  <xacro:property name="upper_arm_length" value="0.20789"/>
+  <!-- Upper arm: horizontal segment from elbow to feeder joint -->
+  <!-- CAD: elbow at X~-5, extends to X~158 = ~163mm -->
+  <xacro:property name="upper_arm_length" value="0.163"/>
   <xacro:property name="upper_arm_radius" value="0.022"/>
-  <xacro:property name="feeder_length" value="0.15965"/>
+  <!-- Feeder: from feeder joint to end effector -->
+  <!-- CAD: feeder joint at X~158, extends to X~343 = ~185mm -->
+  <xacro:property name="feeder_length" value="0.185"/>
   <xacro:property name="feeder_radius" value="0.018"/>
   <!-- Motor housing dimensions (Dynamixel XM430) -->
@@ -25,12 +36,9 @@
   <xacro:property name="motor_height" value="0.0466"/>
   <xacro:property name="motor_depth" value="0.034"/>
-  <!-- Joint limits (radians) - from paper Figure 2 -->
-  <!-- Base Y:   -175 to +175 deg -->
-  <!-- Lower Z:  -90 to +90 deg   -->
-  <!-- Upper Z:  -120 to +75 deg  -->
-  <!-- Feeder:   -90 to +115 deg  -->
   <!-- XM430-W350R specs -->
-  <xacro:property name="max_velocity" value="4.8172"/>   <!-- ~46 RPM -->
-  <xacro:property name="max_effort" value="4.1"/>         <!-- Nm stall torque -->
+  <xacro:property name="max_velocity" value="4.8172"/>
+  <xacro:property name="max_effort" value="4.1"/>
+  <!-- Mesh file path prefix -->
+  <xacro:property name="mesh_path" value="package://feeding_robot/meshes"/>
   <!-- Use mesh files if available, otherwise use primitives -->
   <xacro:arg name="use_meshes" default="false"/>
@@ -44,18 +52,38 @@
   </joint>
   <!-- ==================== BASE LINK ==================== -->
+  <!-- Contains the fixed base platform (CAD solids 59-63) -->
   <link name="base_link">
-    <visual>
-      <geometry>
-        <cylinder radius="${base_radius}" length="${base_height}"/>
-      </geometry>
-      <origin xyz="0 0 ${base_height/2}" rpy="0 0 0"/>
-      <material name="dark_grey"/>
-    </visual>
-    <collision>
-      <geometry>
-        <cylinder radius="${base_radius}" length="${base_height}"/>
-      </geometry>
-      <origin xyz="0 0 ${base_height/2}" rpy="0 0 0"/>
-    </collision>
+    <xacro:if value="${use_meshes}">
+      <visual>
+        <geometry>
+          <mesh filename="${mesh_path}/visual/feeding_robot_full.stl" scale="0.001 0.001 0.001"/>
+        </geometry>
+        <!-- Offset to align CAD origin with URDF origin -->
+        <!-- CAD base center is at approximately X=-25, Y=0, Z=-25 mm -->
+        <origin xyz="0.025 0.0 0.025" rpy="0 0 0"/>
+        <material name="light_grey"/>
+      </visual>
+      <collision>
+        <geometry>
+          <mesh filename="${mesh_path}/collision/feeding_robot_full.stl" scale="0.001 0.001 0.001"/>
+        </geometry>
+        <origin xyz="0.025 0.0 0.025" rpy="0 0 0"/>
+      </collision>
+    </xacro:if>
+    <xacro:unless value="${use_meshes}">
+      <visual>
+        <geometry>
+          <cylinder radius="${base_radius}" length="${base_height}"/>
+        </geometry>
+        <origin xyz="0 0 ${base_height/2}" rpy="0 0 0"/>
+        <material name="dark_grey"/>
+      </visual>
+      <collision>
+        <geometry>
+          <cylinder radius="${base_radius}" length="${base_height}"/>
+        </geometry>
+        <origin xyz="0 0 ${base_height/2}" rpy="0 0 0"/>
+      </collision>
+    </xacro:unless>
     <inertial>
       <mass value="0.8"/>
@@ -78,17 +106,19 @@
   <!-- ==================== TURNTABLE LINK ==================== -->
   <link name="turntable_link">
-    <visual>
-      <geometry>
-        <cylinder radius="${turntable_radius}" length="${turntable_height}"/>
-      </geometry>
-      <origin xyz="0 0 ${turntable_height/2}" rpy="0 0 0"/>
-      <material name="blue"/>
-    </visual>
-    <collision>
-      <geometry>
-        <cylinder radius="${turntable_radius}" length="${turntable_height}"/>
-      </geometry>
-      <origin xyz="0 0 ${turntable_height/2}" rpy="0 0 0"/>
-    </collision>
+    <xacro:unless value="${use_meshes}">
+      <visual>
+        <geometry>
+          <cylinder radius="${turntable_radius}" length="${turntable_height}"/>
+        </geometry>
+        <origin xyz="0 0 ${turntable_height/2}" rpy="0 0 0"/>
+        <material name="blue"/>
+      </visual>
+      <collision>
+        <geometry>
+          <cylinder radius="${turntable_radius}" length="${turntable_height}"/>
+        </geometry>
+        <origin xyz="0 0 ${turntable_height/2}" rpy="0 0 0"/>
+      </collision>
+    </xacro:unless>
     <inertial>
       <mass value="0.3"/>
@@ -100,18 +130,21 @@
   <!-- ==================== SHOULDER RISER ==================== -->
   <!-- Vertical column from turntable to shoulder joint -->
+  <!-- CAD: motor housings stack from Z~88mm to Z~134mm -->
   <link name="shoulder_riser_link">
-    <visual>
-      <geometry>
-        <box size="0.04 0.04 ${shoulder_height}"/>
-      </geometry>
-      <origin xyz="0 0 ${shoulder_height/2}" rpy="0 0 0"/>
-      <material name="light_grey"/>
-    </visual>
-    <collision>
-      <geometry>
-        <box size="0.04 0.04 ${shoulder_height}"/>
-      </geometry>
-      <origin xyz="0 0 ${shoulder_height/2}" rpy="0 0 0"/>
-    </collision>
+    <xacro:unless value="${use_meshes}">
+      <visual>
+        <geometry>
+          <box size="0.04 0.04 ${shoulder_height}"/>
+        </geometry>
+        <origin xyz="0 0 ${shoulder_height/2}" rpy="0 0 0"/>
+        <material name="light_grey"/>
+      </visual>
+      <collision>
+        <geometry>
+          <box size="0.04 0.04 ${shoulder_height}"/>
+        </geometry>
+        <origin xyz="0 0 ${shoulder_height/2}" rpy="0 0 0"/>
+      </collision>
+    </xacro:unless>
     <inertial>
       <mass value="0.35"/>
@@ -138,39 +171,43 @@
   </joint>
   <!-- ==================== LOWER ARM LINK ==================== -->
+  <!-- Vertical arm segment going upward (CAD: Z ~134 to ~338mm) -->
   <link name="lower_arm_link">
-    <!-- Motor housing at joint -->
-    <visual name="lower_motor">
-      <geometry>
-        <box size="${motor_width} ${motor_depth} ${motor_height}"/>
-      </geometry>
-      <origin xyz="0 0 ${motor_height/2}" rpy="0 0 0"/>
-      <material name="black"/>
-    </visual>
-    <!-- Arm segment -->
-    <visual name="lower_arm">
-      <geometry>
-        <cylinder radius="${lower_arm_radius}" length="${lower_arm_length}"/>
-      </geometry>
-      <origin xyz="${lower_arm_length/2 + motor_width/2} 0 0" rpy="0 ${pi/2} 0"/>
-      <material name="red"/>
-    </visual>
-    <collision>
-      <geometry>
-        <box size="${lower_arm_length + motor_width} ${motor_depth} ${motor_height}"/>
-      </geometry>
-      <origin xyz="${lower_arm_length/2} 0 0" rpy="0 0 0"/>
-    </collision>
+    <xacro:unless value="${use_meshes}">
+      <!-- Motor housing at joint -->
+      <visual name="lower_motor">
+        <geometry>
+          <box size="${motor_width} ${motor_depth} ${motor_height}"/>
+        </geometry>
+        <origin xyz="0 0 ${motor_height/2}" rpy="0 0 0"/>
+        <material name="black"/>
+      </visual>
+      <!-- Arm segment -->
+      <visual name="lower_arm">
+        <geometry>
+          <cylinder radius="${lower_arm_radius}" length="${lower_arm_length}"/>
+        </geometry>
+        <origin xyz="0 0 ${lower_arm_length/2 + motor_height/2}" rpy="0 0 0"/>
+        <material name="red"/>
+      </visual>
+      <collision>
+        <geometry>
+          <box size="${motor_width + 0.01} ${motor_depth + 0.01} ${lower_arm_length + motor_height}"/>
+        </geometry>
+        <origin xyz="0 0 ${(lower_arm_length + motor_height)/2}" rpy="0 0 0"/>
+      </collision>
+    </xacro:unless>
     <inertial>
       <mass value="0.4"/>
-      <origin xyz="${lower_arm_length/2} 0 0" rpy="0 0 0"/>
-      <inertia ixx="0.0003" ixy="0.0" ixz="0.0"
-               iyy="0.002" iyz="0.0" izz="0.002"/>
+      <origin xyz="0 0 ${lower_arm_length/2}" rpy="0 0 0"/>
+      <inertia ixx="0.002" ixy="0.0" ixz="0.0"
+               iyy="0.002" iyz="0.0" izz="0.0003"/>
     </inertial>
   </link>
   <!-- ==================== UPPER Z JOINT (Elbow Pitch) ==================== -->
+  <!-- At the top of the vertical arm, transitions to horizontal -->
   <joint name="upper_z_joint" type="revolute">
     <parent link="lower_arm_link"/>
     <child link="upper_arm_link"/>
-    <origin xyz="${lower_arm_length + motor_width/2} 0 0" rpy="0 0 0"/>
+    <origin xyz="0 0 ${lower_arm_length}" rpy="0 0 0"/>
     <axis xyz="0 1 0"/>
     <limit lower="${-120.0 * pi / 180.0}" upper="${75.0 * pi / 180.0}"
@@ -179,27 +216,30 @@
   </joint>
   <!-- ==================== UPPER ARM LINK ==================== -->
+  <!-- Horizontal arm segment (CAD: extends in X from ~-5 to ~158mm) -->
   <link name="upper_arm_link">
-    <!-- Motor housing at joint -->
-    <visual name="upper_motor">
-      <geometry>
-        <box size="${motor_width} ${motor_depth} ${motor_height}"/>
-      </geometry>
-      <origin xyz="0 0 0" rpy="0 0 0"/>
-      <material name="black"/>
-    </visual>
-    <!-- Arm segment -->
-    <visual name="upper_arm">
-      <geometry>
-        <cylinder radius="${upper_arm_radius}" length="${upper_arm_length}"/>
-      </geometry>
-      <origin xyz="${upper_arm_length/2 + motor_width/2} 0 0" rpy="0 ${pi/2} 0"/>
-      <material name="blue"/>
-    </visual>
-    <collision>
-      <geometry>
-        <box size="${upper_arm_length + motor_width} ${motor_depth} ${motor_height}"/>
-      </geometry>
-      <origin xyz="${upper_arm_length/2} 0 0" rpy="0 0 0"/>
-    </collision>
+    <xacro:unless value="${use_meshes}">
+      <!-- Motor housing at joint -->
+      <visual name="upper_motor">
+        <geometry>
+          <box size="${motor_width} ${motor_depth} ${motor_height}"/>
+        </geometry>
+        <origin xyz="0 0 0" rpy="0 0 0"/>
+        <material name="black"/>
+      </visual>
+      <!-- Arm segment extending horizontally -->
+      <visual name="upper_arm">
+        <geometry>
+          <cylinder radius="${upper_arm_radius}" length="${upper_arm_length}"/>
+        </geometry>
+        <origin xyz="${upper_arm_length/2 + motor_width/2} 0 0" rpy="0 ${pi/2} 0"/>
+        <material name="blue"/>
+      </visual>
+      <collision>
+        <geometry>
+          <box size="${upper_arm_length + motor_width} ${motor_depth} ${motor_height}"/>
+        </geometry>
+        <origin xyz="${upper_arm_length/2} 0 0" rpy="0 0 0"/>
+      </collision>
+    </xacro:unless>
     <inertial>
       <mass value="0.35"/>
@@ -220,35 +260,38 @@
   </joint>
   <!-- ==================== FEEDER LINK (End Effector) ==================== -->
+  <!-- CAD: extends from X~158 to X~343mm with sensors and fork -->
   <link name="feeder_link">
-    <!-- Motor housing -->
-    <visual name="feeder_motor">
-      <geometry>
-        <box size="${motor_width} ${motor_depth} ${motor_height}"/>
-      </geometry>
-      <origin xyz="0 0 0" rpy="0 0 0"/>
-      <material name="black"/>
-    </visual>
-    <!-- Fork/spoon shaft -->
-    <visual name="feeder_shaft">
-      <geometry>
-        <cylinder radius="${feeder_radius}" length="${feeder_length}"/>
-      </geometry>
-      <origin xyz="${feeder_length/2 + motor_width/2} 0 0" rpy="0 ${pi/2} 0"/>
-      <material name="orange"/>
-    </visual>
-    <!-- Fork tines / spoon head -->
-    <visual name="feeder_head">
-      <geometry>
-        <box size="0.04 0.03 0.005"/>
-      </geometry>
-      <origin xyz="${feeder_length + motor_width/2 + 0.02} 0 0" rpy="0 0 0"/>
-      <material name="light_grey"/>
-    </visual>
-    <collision>
-      <geometry>
-        <box size="${feeder_length + 0.04} ${motor_depth} ${motor_height}"/>
-      </geometry>
-      <origin xyz="${feeder_length/2 + 0.02} 0 0" rpy="0 0 0"/>
-    </collision>
+    <xacro:unless value="${use_meshes}">
+      <!-- Motor housing -->
+      <visual name="feeder_motor">
+        <geometry>
+          <box size="${motor_width} ${motor_depth} ${motor_height}"/>
+        </geometry>
+        <origin xyz="0 0 0" rpy="0 0 0"/>
+        <material name="black"/>
+      </visual>
+      <!-- Fork/spoon shaft -->
+      <visual name="feeder_shaft">
+        <geometry>
+          <cylinder radius="${feeder_radius}" length="${feeder_length}"/>
+        </geometry>
+        <origin xyz="${feeder_length/2 + motor_width/2} 0 0" rpy="0 ${pi/2} 0"/>
+        <material name="orange"/>
+      </visual>
+      <!-- Fork tines / spoon head -->
+      <visual name="feeder_head">
+        <geometry>
+          <box size="0.04 0.03 0.005"/>
+        </geometry>
+        <origin xyz="${feeder_length + motor_width/2 + 0.02} 0 0" rpy="0 0 0"/>
+        <material name="light_grey"/>
+      </visual>
+      <collision>
+        <geometry>
+          <box size="${feeder_length + 0.04} ${motor_depth} ${motor_height}"/>
+        </geometry>
+        <origin xyz="${feeder_length/2 + 0.02} 0 0" rpy="0 0 0"/>
+      </collision>
+    </xacro:unless>
     <inertial>
       <mass value="0.25"/>
@@ -294,5 +337,4 @@
     <parent link="camera_link"/>
     <child link="camera_optical_frame"/>
-    <!-- Standard ROS camera optical frame convention: Z forward, X right, Y down -->
     <origin xyz="0 0 0" rpy="${-pi/2} 0 ${-pi/2}"/>
   </joint>
@@ -323,5 +365,4 @@
   </joint>
   <!-- ==================== LOAD CELL (HX711) ==================== -->
-  <!-- Conceptual frame at the fork tip for force sensing -->
   <link name="load_cell_frame"/>
   <joint name="load_cell_joint" type="fixed">
