Commit message: Initial commit

File: feeding_robot/description/feeding_robot_core.xacro (robot description, xacro)
@@ -3,45 +3,39 @@
   <!-- ============================================================ -->
   <!-- Adaptive Feeding Robot - 4 DOF Open Manipulator               -->
-  <!-- Based on: Sadeghi Esfahlani et al. (2025)                    -->
-  <!-- CAD source: Auto Feeder SSE v222.step                        -->
+  <!-- CAD: Auto Feeder SSE v222.step                                -->
   <!-- Joints: Base Y, Lower Z, Upper Z, Feeder                     -->
   <!-- Actuators: 4x Dynamixel XM430-W350R                          -->
+  <!--                                                               -->
+  <!-- CAD coordinate system: Z up, X horizontal (arm extends +X)   -->
+  <!-- Assembly bounds (mm): X[-75,343] Y[-55,56] Z[-25,425]        -->
   <!-- ============================================================ -->
   <!-- ==================== PARAMETERS ==================== -->
-  <!-- Dimensions (metres) - measured from CAD bounding boxes -->
-  <!-- CAD assembly: X: -75 to 343mm, Y: -55 to 56mm, Z: -25 to 425mm -->
-  <!-- Base center at approximately X=-25, Y=0, Z=0 in CAD coords -->
-  <xacro:property name="base_height" value="0.088"/>
-  <xacro:property name="base_radius" value="0.060"/>
-  <xacro:property name="turntable_height" value="0.050"/>
-  <xacro:property name="turntable_radius" value="0.045"/>
-  <!-- Shoulder height: from base top to lower_z_joint axis -->
-  <!-- CAD: first motor (solid_000) center at Z=111.7mm, base top ~88mm -->
-  <!-- Joint axis at approximately Z=134mm from ground -->
-  <xacro:property name="shoulder_height" value="0.134"/>
-  <!-- Lower arm: vertical segment from shoulder to elbow -->
-  <!-- CAD: shoulder at Z~134mm, top of vertical arm at Z~338mm = 204mm -->
-  <xacro:property name="lower_arm_length" value="0.204"/>
-  <xacro:property name="lower_arm_radius" value="0.025"/>
-  <!-- Upper arm: horizontal segment from elbow to feeder joint -->
-  <!-- CAD: elbow at X~-5, extends to X~158 = ~163mm -->
-  <xacro:property name="upper_arm_length" value="0.163"/>
-  <xacro:property name="upper_arm_radius" value="0.022"/>
-  <!-- Feeder: from feeder joint to end effector -->
-  <!-- CAD: feeder joint at X~158, extends to X~343 = ~185mm -->
-  <xacro:property name="feeder_length" value="0.185"/>
-  <xacro:property name="feeder_radius" value="0.018"/>
-  <!-- Motor housing dimensions (Dynamixel XM430) -->
-  <xacro:property name="motor_width" value="0.0286"/>
-  <xacro:property name="motor_height" value="0.0466"/>
-  <xacro:property name="motor_depth" value="0.034"/>
-  <!-- XM430-W350R specs -->
+  <!-- Joint positions in CAD coordinates (mm), converted to metres -->
+  <!-- These are derived from the bounding box analysis of grouped solids -->
+  <!-- Base Y joint: at top of base platform, Z=88mm -->
+  <xacro:property name="base_top_z" value="0.088"/>
+  <!-- Lower Z joint (shoulder): at Z=131mm, X=-16mm -->
+  <!-- This is where the shoulder motor stack meets the vertical arm -->
+  <xacro:property name="shoulder_joint_z" value="0.131"/>
+  <!-- Upper Z joint (elbow): at top of vertical arm, Z=331mm, X=-5mm -->
+  <!-- Transition from vertical to horizontal arm -->
+  <xacro:property name="elbow_joint_z" value="0.331"/>
+  <xacro:property name="lower_arm_length" value="${elbow_joint_z - shoulder_joint_z}"/>
+  <!-- Feeder joint (wrist): at X=194mm from CAD origin, Z=351mm -->
+  <!-- Where the horizontal arm meets the feeder end effector -->
+  <xacro:property name="upper_arm_length" value="0.199"/>
+  <!-- Feeder length to tip -->
+  <xacro:property name="feeder_length" value="0.148"/>
+  <!-- Motor specs: Dynamixel XM430-W350R -->
   <xacro:property name="max_velocity" value="4.8172"/>
   <xacro:property name="max_effort" value="4.1"/>
-  <!-- Mesh file path prefix -->
-  <xacro:property name="mesh_path" value="package://feeding_robot/meshes"/>
-  <!-- Use mesh files if available, otherwise use primitives -->
+  <!-- Mesh file paths -->
+  <xacro:property name="mesh_vis" value="package://feeding_robot/meshes/visual"/>
+  <xacro:property name="mesh_col" value="package://feeding_robot/meshes/collision"/>
+  <!-- Switch between mesh and primitive visuals -->
   <xacro:arg name="use_meshes" default="false"/>
   <xacro:property name="use_meshes" value="$(arg use_meshes)"/>
+  <!-- STL scale: CAD is in mm, URDF uses metres -->
+  <xacro:property name="stl_scale" value="0.001 0.001 0.001"/>
   <!-- ==================== WORLD LINK ==================== -->
   <link name="world"/>
@@ -52,51 +46,49 @@
   </joint>
   <!-- ==================== BASE LINK ==================== -->
-  <!-- Contains the fixed base platform (CAD solids 59-63) -->
+  <!-- CAD solids 59-63: base platform, Z[-25, 88]mm -->
   <link name="base_link">
     <xacro:if value="${use_meshes}">
       <visual>
         <geometry>
-          <mesh filename="${mesh_path}/visual/feeding_robot_full.stl" scale="0.001 0.001 0.001"/>
-        </geometry>
-        <!-- Offset to align CAD origin with URDF origin -->
-        <!-- CAD base center is at approximately X=-25, Y=0, Z=-25 mm -->
-        <origin xyz="0.025 0.0 0.025" rpy="0 0 0"/>
-        <material name="light_grey"/>
-      </visual>
-      <collision>
-        <geometry>
-          <mesh filename="${mesh_path}/collision/feeding_robot_full.stl" scale="0.001 0.001 0.001"/>
-        </geometry>
-        <origin xyz="0.025 0.0 0.025" rpy="0 0 0"/>
-      </collision>
-    </xacro:if>
-    <xacro:unless value="${use_meshes}">
-      <visual>
-        <geometry>
-          <cylinder radius="${base_radius}" length="${base_height}"/>
-        </geometry>
-        <origin xyz="0 0 ${base_height/2}" rpy="0 0 0"/>
+          <mesh filename="${mesh_vis}/base_link.stl" scale="${stl_scale}"/>
+        </geometry>
+        <!-- CAD origin is at world origin, no offset needed -->
+        <origin xyz="0 0 0" rpy="0 0 0"/>
+      </visual>
+      <collision>
+        <geometry>
+          <mesh filename="${mesh_col}/base_link.stl" scale="${stl_scale}"/>
+        </geometry>
+        <origin xyz="0 0 0" rpy="0 0 0"/>
+      </collision>
+    </xacro:if>
+    <xacro:unless value="${use_meshes}">
+      <visual>
+        <geometry>
+          <cylinder radius="0.060" length="${base_top_z}"/>
+        </geometry>
+        <origin xyz="0 0 ${base_top_z/2}" rpy="0 0 0"/>
         <material name="dark_grey"/>
       </visual>
       <collision>
         <geometry>
-          <cylinder radius="${base_radius}" length="${base_height}"/>
-        </geometry>
-        <origin xyz="0 0 ${base_height/2}" rpy="0 0 0"/>
+          <cylinder radius="0.060" length="${base_top_z}"/>
+        </geometry>
+        <origin xyz="0 0 ${base_top_z/2}" rpy="0 0 0"/>
       </collision>
     </xacro:unless>
     <inertial>
       <mass value="0.8"/>
-      <origin xyz="0 0 ${base_height/2}" rpy="0 0 0"/>
-      <inertia ixx="0.001" ixy="0.0" ixz="0.0"
-               iyy="0.001" iyz="0.0" izz="0.001"/>
+      <origin xyz="-0.034 0 0.032" rpy="0 0 0"/>
+      <inertia ixx="0.002" ixy="0.0" ixz="0.0"
+               iyy="0.002" iyz="0.0" izz="0.001"/>
     </inertial>
   </link>
   <!-- ==================== BASE Y JOINT (Yaw) ==================== -->
-  <!-- Rotates the entire arm around the vertical axis -->
+  <!-- At the top of the base platform, rotates around vertical Z axis -->
   <joint name="base_y_joint" type="revolute">
     <parent link="base_link"/>
-    <child link="turntable_link"/>
-    <origin xyz="0 0 ${base_height}" rpy="0 0 0"/>
+    <child link="shoulder_link"/>
+    <origin xyz="0 0 ${base_top_z}" rpy="0 0 0"/>
     <axis xyz="0 0 1"/>
     <limit lower="${-175.0 * pi / 180.0}" upper="${175.0 * pi / 180.0}"
@@ -104,65 +96,51 @@
     <dynamics damping="0.5" friction="0.1"/>
   </joint>
-  <!-- ==================== TURNTABLE LINK ==================== -->
-  <link name="turntable_link">
-    <xacro:unless value="${use_meshes}">
-      <visual>
-        <geometry>
-          <cylinder radius="${turntable_radius}" length="${turntable_height}"/>
-        </geometry>
-        <origin xyz="0 0 ${turntable_height/2}" rpy="0 0 0"/>
-        <material name="blue"/>
-      </visual>
-      <collision>
-        <geometry>
-          <cylinder radius="${turntable_radius}" length="${turntable_height}"/>
-        </geometry>
-        <origin xyz="0 0 ${turntable_height/2}" rpy="0 0 0"/>
-      </collision>
-    </xacro:unless>
-    <inertial>
-      <mass value="0.3"/>
-      <origin xyz="0 0 ${turntable_height/2}" rpy="0 0 0"/>
-      <inertia ixx="0.0005" ixy="0.0" ixz="0.0"
-               iyy="0.0005" iyz="0.0" izz="0.0003"/>
-    </inertial>
-  </link>
-  <!-- ==================== SHOULDER RISER ==================== -->
-  <!-- Vertical column from turntable to shoulder joint -->
-  <!-- CAD: motor housings stack from Z~88mm to Z~134mm -->
-  <link name="shoulder_riser_link">
-    <xacro:unless value="${use_meshes}">
-      <visual>
-        <geometry>
-          <box size="0.04 0.04 ${shoulder_height}"/>
-        </geometry>
-        <origin xyz="0 0 ${shoulder_height/2}" rpy="0 0 0"/>
+  <!-- ==================== SHOULDER LINK ==================== -->
+  <!-- CAD solids 0-10,58: motor stack, Z[81, 132]mm -->
+  <!-- This link sits on top of the base and contains the shoulder motors -->
+  <link name="shoulder_link">
+    <xacro:if value="${use_meshes}">
+      <visual>
+        <geometry>
+          <mesh filename="${mesh_vis}/shoulder_link.stl" scale="${stl_scale}"/>
+        </geometry>
+        <!-- Offset: shift mesh so joint position (CAD X=-25,Y=0,Z=88) is at link origin -->
+        <origin xyz="0.025 0 -0.088" rpy="0 0 0"/>
+      </visual>
+      <collision>
+        <geometry>
+          <mesh filename="${mesh_col}/shoulder_link.stl" scale="${stl_scale}"/>
+        </geometry>
+        <origin xyz="0.025 0 -0.088" rpy="0 0 0"/>
+      </collision>
+    </xacro:if>
+    <xacro:unless value="${use_meshes}">
+      <visual>
+        <geometry>
+          <box size="0.105 0.105 0.051"/>
+        </geometry>
+        <origin xyz="0 0 ${(shoulder_joint_z - base_top_z)/2}" rpy="0 0 0"/>
         <material name="light_grey"/>
       </visual>
       <collision>
         <geometry>
-          <box size="0.04 0.04 ${shoulder_height}"/>
-        </geometry>
-        <origin xyz="0 0 ${shoulder_height/2}" rpy="0 0 0"/>
-      </collision>
-    </xacro:unless>
-    <inertial>
-      <mass value="0.35"/>
-      <origin xyz="0 0 ${shoulder_height/2}" rpy="0 0 0"/>
+          <box size="0.105 0.105 0.051"/>
+        </geometry>
+        <origin xyz="0 0 ${(shoulder_joint_z - base_top_z)/2}" rpy="0 0 0"/>
+      </collision>
+    </xacro:unless>
+    <inertial>
+      <mass value="0.5"/>
+      <origin xyz="0 0 ${(shoulder_joint_z - base_top_z)/2}" rpy="0 0 0"/>
       <inertia ixx="0.001" ixy="0.0" ixz="0.0"
-               iyy="0.001" iyz="0.0" izz="0.0002"/>
-    </inertial>
-  </link>
-  <joint name="turntable_to_shoulder_riser" type="fixed">
-    <parent link="turntable_link"/>
-    <child link="shoulder_riser_link"/>
-    <origin xyz="0 0 ${turntable_height}" rpy="0 0 0"/>
-  </joint>
+               iyy="0.001" iyz="0.0" izz="0.001"/>
+    </inertial>
+  </link>
   <!-- ==================== LOWER Z JOINT (Shoulder Pitch) ==================== -->
-  <!-- Rotates the lower arm up/down -->
+  <!-- At the top of the shoulder motor stack, Z=131mm -->
   <joint name="lower_z_joint" type="revolute">
-    <parent link="shoulder_riser_link"/>
+    <parent link="shoulder_link"/>
     <child link="lower_arm_link"/>
-    <origin xyz="0 0 ${shoulder_height}" rpy="0 0 0"/>
+    <origin xyz="0 0 ${shoulder_joint_z - base_top_z}" rpy="0 0 0"/>
     <axis xyz="0 1 0"/>
     <limit lower="${-90.0 * pi / 180.0}" upper="${90.0 * pi / 180.0}"
@@ -171,39 +149,53 @@
   </joint>
   <!-- ==================== LOWER ARM LINK ==================== -->
-  <!-- Vertical arm segment going upward (CAD: Z ~134 to ~338mm) -->
+  <!-- CAD solids 11-21,23-26: vertical arm segment, Z[127, 331]mm -->
+  <!-- Goes upward 200mm from shoulder to elbow -->
   <link name="lower_arm_link">
-    <xacro:unless value="${use_meshes}">
-      <!-- Motor housing at joint -->
-      <visual name="lower_motor">
-        <geometry>
-          <box size="${motor_width} ${motor_depth} ${motor_height}"/>
-        </geometry>
-        <origin xyz="0 0 ${motor_height/2}" rpy="0 0 0"/>
+    <xacro:if value="${use_meshes}">
+      <visual>
+        <geometry>
+          <mesh filename="${mesh_vis}/lower_arm_link.stl" scale="${stl_scale}"/>
+        </geometry>
+        <!-- Offset: shift mesh so joint position (CAD X=-16,Y=0,Z=131) is at link origin -->
+        <origin xyz="0.016 0 -0.131" rpy="0 0 0"/>
+      </visual>
+      <collision>
+        <geometry>
+          <mesh filename="${mesh_col}/lower_arm_link.stl" scale="${stl_scale}"/>
+        </geometry>
+        <origin xyz="0.016 0 -0.131" rpy="0 0 0"/>
+      </collision>
+    </xacro:if>
+    <xacro:unless value="${use_meshes}">
+      <visual>
+        <geometry>
+          <cylinder radius="0.020" length="${lower_arm_length}"/>
+        </geometry>
+        <origin xyz="0 0 ${lower_arm_length/2}" rpy="0 0 0"/>
+        <material name="red"/>
+      </visual>
+      <visual>
+        <geometry>
+          <box size="0.029 0.034 0.047"/>
+        </geometry>
+        <origin xyz="0 0 0.023" rpy="0 0 0"/>
         <material name="black"/>
       </visual>
-      <!-- Arm segment -->
-      <visual name="lower_arm">
-        <geometry>
-          <cylinder radius="${lower_arm_radius}" length="${lower_arm_length}"/>
-        </geometry>
-        <origin xyz="0 0 ${lower_arm_length/2 + motor_height/2}" rpy="0 0 0"/>
-        <material name="red"/>
-      </visual>
-      <collision>
-        <geometry>
-          <box size="${motor_width + 0.01} ${motor_depth + 0.01} ${lower_arm_length + motor_height}"/>
-        </geometry>
-        <origin xyz="0 0 ${(lower_arm_length + motor_height)/2}" rpy="0 0 0"/>
-      </collision>
-    </xacro:unless>
-    <inertial>
-      <mass value="0.4"/>
+      <collision>
+        <geometry>
+          <box size="0.029 0.045 ${lower_arm_length}"/>
+        </geometry>
+        <origin xyz="0 0 ${lower_arm_length/2}" rpy="0 0 0"/>
+      </collision>
+    </xacro:unless>
+    <inertial>
+      <mass value="0.5"/>
       <origin xyz="0 0 ${lower_arm_length/2}" rpy="0 0 0"/>
-      <inertia ixx="0.002" ixy="0.0" ixz="0.0"
-               iyy="0.002" iyz="0.0" izz="0.0003"/>
+      <inertia ixx="0.003" ixy="0.0" ixz="0.0"
+               iyy="0.003" iyz="0.0" izz="0.0003"/>
     </inertial>
   </link>
   <!-- ==================== UPPER Z JOINT (Elbow Pitch) ==================== -->
-  <!-- At the top of the vertical arm, transitions to horizontal -->
+  <!-- At the top of the vertical arm, Z=331mm, transition to horizontal -->
   <joint name="upper_z_joint" type="revolute">
     <parent link="lower_arm_link"/>
@@ -216,26 +208,40 @@
   </joint>
   <!-- ==================== UPPER ARM LINK ==================== -->
-  <!-- Horizontal arm segment (CAD: extends in X from ~-5 to ~158mm) -->
+  <!-- CAD solids 22,27-52: horizontal arm, X[-28, 198]mm Z[331, 386]mm -->
+  <!-- Extends horizontally ~200mm from elbow to wrist -->
   <link name="upper_arm_link">
-    <xacro:unless value="${use_meshes}">
-      <!-- Motor housing at joint -->
-      <visual name="upper_motor">
-        <geometry>
-          <box size="${motor_width} ${motor_depth} ${motor_height}"/>
+    <xacro:if value="${use_meshes}">
+      <visual>
+        <geometry>
+          <mesh filename="${mesh_vis}/upper_arm_link.stl" scale="${stl_scale}"/>
+        </geometry>
+        <!-- Offset: shift mesh so elbow joint (CAD X=-5,Y=0,Z=331) is at link origin -->
+        <origin xyz="0.005 0 -0.331" rpy="0 0 0"/>
+      </visual>
+      <collision>
+        <geometry>
+          <mesh filename="${mesh_col}/upper_arm_link.stl" scale="${stl_scale}"/>
+        </geometry>
+        <origin xyz="0.005 0 -0.331" rpy="0 0 0"/>
+      </collision>
+    </xacro:if>
+    <xacro:unless value="${use_meshes}">
+      <visual>
+        <geometry>
+          <cylinder radius="0.018" length="${upper_arm_length}"/>
+        </geometry>
+        <origin xyz="${upper_arm_length/2} 0 0" rpy="0 ${pi/2} 0"/>
+        <material name="blue"/>
+      </visual>
+      <visual>
+        <geometry>
+          <box size="0.029 0.034 0.047"/>
         </geometry>
         <origin xyz="0 0 0" rpy="0 0 0"/>
         <material name="black"/>
       </visual>
-      <!-- Arm segment extending horizontally -->
-      <visual name="upper_arm">
-        <geometry>
-          <cylinder radius="${upper_arm_radius}" length="${upper_arm_length}"/>
-        </geometry>
-        <origin xyz="${upper_arm_length/2 + motor_width/2} 0 0" rpy="0 ${pi/2} 0"/>
-        <material name="blue"/>
-      </visual>
-      <collision>
-        <geometry>
-          <box size="${upper_arm_length + motor_width} ${motor_depth} ${motor_height}"/>
+      <collision>
+        <geometry>
+          <box size="${upper_arm_length} 0.045 0.055"/>
         </geometry>
         <origin xyz="${upper_arm_length/2} 0 0" rpy="0 0 0"/>
@@ -243,15 +249,16 @@
     </xacro:unless>
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
File: feeding_robot/description/gazebo_plugins.xacro (robot description, xacro)
@@ -5,8 +5,5 @@
     <material>Gazebo/DarkGrey</material>
   </gazebo>
-  <gazebo reference="turntable_link">
-    <material>Gazebo/Blue</material>
-  </gazebo>
-  <gazebo reference="shoulder_riser_link">
+  <gazebo reference="shoulder_link">
     <material>Gazebo/Grey</material>
   </gazebo>

Commit message: update

File: feeding_robot/description/feeding_robot_core.xacro (robot description, xacro)
@@ -272,5 +272,5 @@
       <visual>
         <geometry>
-          <mesh filename="${mesh_vis}/feeder_link.stl" scale="${stl_scale}"/>
+          <mesh filename="${mesh_vis}/frontface.stl" scale="${stl_scale}"/>
         </geometry>
         <!-- Offset: shift mesh so wrist joint (CAD X=194,Y=0,Z=351) is at link origin -->
@@ -331,11 +331,10 @@
     <visual>
       <geometry>
-        <box size="0.025 0.024 0.009"/>
-      </geometry>
-      <material name="green"/>
+        <mesh filename="${mesh_vis}/camera.stl" scale="${stl_scale}"/>
+      </geometry>
     </visual>
     <collision>
       <geometry>
-        <box size="0.025 0.024 0.009"/>
+        <mesh filename="${mesh_vis}/camera.stl" scale="${stl_scale}"/>
       </geometry>
     </collision>
@@ -361,11 +360,10 @@
     <visual>
       <geometry>
-        <box size="0.045 0.020 0.015"/>
-      </geometry>
-      <material name="blue"/>
+        <mesh filename="${mesh_vis}/sonar.stl" scale="${stl_scale}"/>
+      </geometry>
     </visual>
     <collision>
       <geometry>
-        <box size="0.045 0.020 0.015"/>
+        <mesh filename="${mesh_vis}/sonar.stl" scale="${stl_scale}"/>
       </geometry>
     </collision>
@@ -382,5 +380,21 @@
   </joint>
   <!-- ==================== LOAD CELL (HX711) ==================== -->
-  <link name="load_cell_frame"/>
+  <link name="load_cell_frame">
+    <visual>
+      <geometry>
+        <mesh filename="${mesh_vis}/forceSensor.stl" scale="${stl_scale}"/>
+      </geometry>
+    </visual>
+    <collision>
+      <geometry>
+        <mesh filename="${mesh_vis}/forceSensor.stl" scale="${stl_scale}"/>
+      </geometry>
+    </collision>
+    <inertial>
+      <mass value="0.010"/>
+      <inertia ixx="0.000001" ixy="0.0" ixz="0.0"
+               iyy="0.000001" iyz="0.0" izz="0.000001"/>
+    </inertial>
+  </link>
   <joint name="load_cell_joint" type="fixed">
     <parent link="feeder_link"/>

Commit message: update

File: feeding_robot/description/feeding_robot_core.xacro (robot description, xacro)
@@ -333,4 +333,6 @@
         <mesh filename="${mesh_vis}/camera.stl" scale="${stl_scale}"/>
       </geometry>
+      <!-- CAD origin offset minus camera_joint offset (0.03, 0, 0.05) -->
+      <origin xyz="${-0.194 - 0.03} 0 ${-0.351 - 0.05}" rpy="0 0 0"/>
     </visual>
     <collision>
@@ -338,4 +340,5 @@
         <mesh filename="${mesh_vis}/camera.stl" scale="${stl_scale}"/>
       </geometry>
+      <origin xyz="${-0.194 - 0.03} 0 ${-0.351 - 0.05}" rpy="0 0 0"/>
     </collision>
     <inertial>
@@ -362,4 +365,6 @@
         <mesh filename="${mesh_vis}/sonar.stl" scale="${stl_scale}"/>
       </geometry>
+      <!-- CAD origin offset minus ultrasonic_joint offset (0.03, 0, -0.04) -->
+      <origin xyz="${-0.194 - 0.03} 0 ${-0.351 + 0.04}" rpy="0 0 0"/>
     </visual>
     <collision>
@@ -367,4 +372,5 @@
         <mesh filename="${mesh_vis}/sonar.stl" scale="${stl_scale}"/>
       </geometry>
+      <origin xyz="${-0.194 - 0.03} 0 ${-0.351 + 0.04}" rpy="0 0 0"/>
     </collision>
     <inertial>
@@ -385,4 +391,6 @@
         <mesh filename="${mesh_vis}/forceSensor.stl" scale="${stl_scale}"/>
       </geometry>
+      <!-- CAD origin offset minus load_cell_joint offset (feeder_length, 0, 0) -->
+      <origin xyz="${-0.194 - feeder_length} 0 -0.351" rpy="0 0 0"/>
     </visual>
     <collision>
@@ -390,4 +398,5 @@
         <mesh filename="${mesh_vis}/forceSensor.stl" scale="${stl_scale}"/>
       </geometry>
+      <origin xyz="${-0.194 - feeder_length} 0 -0.351" rpy="0 0 0"/>
     </collision>
     <inertial>

Commit message: update

File: feeding_robot/description/feeding_robot_core.xacro (robot description, xacro)
@@ -365,6 +365,6 @@
         <mesh filename="${mesh_vis}/sonar.stl" scale="${stl_scale}"/>
       </geometry>
-      <!-- CAD origin offset minus ultrasonic_joint offset (0.03, 0, -0.04) -->
-      <origin xyz="${-0.194 - 0.03} 0 ${-0.351 + 0.04}" rpy="0 0 0"/>
+      <!-- CAD origin offset minus ultrasonic_joint offset; Y shifted from CAD side (116mm) to face -->
+      <origin xyz="${-0.194 - 0.03} -0.116 ${-0.351 + 0.04}" rpy="0 0 0"/>
     </visual>
     <collision>
@@ -372,5 +372,5 @@
         <mesh filename="${mesh_vis}/sonar.stl" scale="${stl_scale}"/>
       </geometry>
-      <origin xyz="${-0.194 - 0.03} 0 ${-0.351 + 0.04}" rpy="0 0 0"/>
+      <origin xyz="${-0.194 - 0.03} -0.116 ${-0.351 + 0.04}" rpy="0 0 0"/>
     </collision>
     <inertial>
