Commit message: update

File: feeding_robot/description/feeding_robot_core.xacro (robot description, xacro)
@@ -411,3 +411,28 @@
     <origin xyz="${feeder_length} 0 0" rpy="0 0 0"/>
   </joint>
+  <!-- ==================== PLATE (fixed in front of robot) ==================== -->
+  <link name="plate_link">
+    <visual>
+      <geometry>
+        <mesh filename="${mesh_vis}/plate_printing.stl"/>
+      </geometry>
+      <origin xyz="0 0 0" rpy="0 0 0"/>
+    </visual>
+    <collision>
+      <geometry>
+        <mesh filename="${mesh_vis}/plate_printing.stl"/>
+      </geometry>
+    </collision>
+    <inertial>
+      <mass value="0.2"/>
+      <inertia ixx="0.001" ixy="0.0" ixz="0.0"
+               iyy="0.001" iyz="0.0" izz="0.001"/>
+    </inertial>
+  </link>
+  <joint name="plate_joint" type="fixed">
+    <parent link="world"/>
+    <child link="plate_link"/>
+    <!-- Plate: below feeder head (arm extends to -X in RViz due to flipped axes) -->
+    <origin xyz="0.25 -0.25 0.050" rpy="0 0 0"/>
+  </joint>
 </robot>

File: ros2_feedbot_ws/src/feeding_robot/description/feeding_robot_core.xacro (robot description, xacro)
@@ -87,11 +87,10 @@
   <!-- ==================== BASE Y JOINT (Yaw) ==================== -->
   <!-- At the top of the base platform, rotates around vertical Z axis -->
-  <joint name="base_y_joint" type="revolute">
+  <joint name="base_y_joint" type="continuous">
     <parent link="base_link"/>
     <child link="shoulder_link"/>
     <origin xyz="0 0 ${base_top_z}" rpy="0 0 0"/>
     <axis xyz="0 0 1"/>
-    <limit lower="${-175.0 * pi / 180.0}" upper="${175.0 * pi / 180.0}"
-           velocity="${max_velocity}" effort="${max_effort}"/>
+    <limit velocity="${max_velocity}" effort="${max_effort}"/>
     <dynamics damping="0.5" friction="0.1"/>
   </joint>

Commit message: update

File: feeding_robot/description/feeding_robot_core.xacro (robot description, xacro)
@@ -434,5 +434,5 @@
     <child link="plate_link"/>
     <!-- Plate: below feeder head (arm extends to -X in RViz due to flipped axes) -->
-    <origin xyz="0.25 -0.25 0.050" rpy="0 0 0"/>
+    <origin xyz="0.3 -0.25 0.0750" rpy="0 0 0"/>
   </joint>
 </robot>
