Commit message: updates

File: ros2_feedbot_ws/src/feedbot_description/urdf/my_robot.urdf.xacro (robot description, xacro)
@@ -190,4 +190,22 @@
   </inertial>
 </link>
+<gazebo reference="base">
+  <material>Gazebo/DarkGrey</material>
+</gazebo>
+<gazebo reference="link1">
+  <material>Gazebo/Orange</material>
+</gazebo>
+<gazebo reference="link2">
+  <material>Gazebo/Orange</material>
+</gazebo>
+<gazebo reference="link3">
+  <material>Gazebo/Orange</material>
+</gazebo>
+<gazebo reference="feeder_head">
+  <material>Gazebo/Grey</material>
+</gazebo>
+<gazebo reference="table_link">
+  <material>Gazebo/Wood</material>
+</gazebo>
 <gazebo reference="plate_link">
   <material>Gazebo/White</material>

Commit message: updates

File: ros2_feedbot_ws/src/feedbot_description/urdf/my_robot.urdf.xacro (robot description, xacro)
@@ -346,10 +346,10 @@
   <parent link="feeder_head"/>
   <child link="camera_link"/>
-<origin xyz="0.08 0 0.14" rpy="-1.57 0 1.57"/>
+<origin xyz="0.02 0 0.03" rpy="0 0 0"/>
 </joint>
 <link name="camera_link">
   <visual>
     <geometry>
-      <box size="0.02 0.02 0.02"/>
+      <box size="0.008 0.008 0.005"/>
     </geometry>
     <material name="black"/>

Commit message: updates

File: ros2_feedbot_ws/src/feedbot_description/urdf/my_robot.urdf.xacro (robot description, xacro)
@@ -362,10 +362,13 @@
 </joint>
 <link name="camera_optical_link"/>
+<!-- ==================== CAMERA SENSOR ==================== -->
 <gazebo reference="camera_link">
   <sensor type="camera" name="camera_sensor">
     <always_on>true</always_on>
     <update_rate>30</update_rate>
-    <camera>
-      <horizontal_fov>1.3962634</horizontal_fov>
+    <visualize>true</visualize>
+    <topic>feeding_robot/camera/image_raw</topic>
+    <camera name="feeding_camera">
+      <horizontal_fov>1.0857</horizontal_fov>
       <image>
         <width>640</width>
@@ -374,8 +377,71 @@
       </image>
       <clip>
-        <near>0.01</near>
-        <far>10</far>
+        <near>0.02</near>
+        <far>5.0</far>
       </clip>
+      <noise>
+        <type>gaussian</type>
+        <mean>0.0</mean>
+        <stddev>0.007</stddev>
+      </noise>
     </camera>
+  </sensor>
+</gazebo>
+<!-- ==================== ULTRASONIC SENSOR ==================== -->
+<!-- HC-SR04: range 2cm - 400cm, beam angle ~15 deg -->
+<joint name="ultrasonic_joint" type="fixed">
+  <parent link="feeder_head"/>
+  <child link="ultrasonic_link"/>
+  <origin xyz="0.02 0 -0.015" rpy="0 0 0"/>
+</joint>
+<link name="ultrasonic_link">
+  <visual>
+    <geometry>
+      <box size="0.01 0.005 0.004"/>
+    </geometry>
+    <material name="blue">
+      <color rgba="0.2 0.2 0.8 1"/>
+    </material>
+  </visual>
+  <inertial>
+    <mass value="0.01"/>
+    <inertia ixx="0.00001" iyy="0.00001" izz="0.00001" ixy="0" ixz="0" iyz="0"/>
+  </inertial>
+</link>
+<gazebo reference="ultrasonic_link">
+  <sensor type="gpu_lidar" name="ultrasonic_sensor">
+    <always_on>true</always_on>
+    <update_rate>20.0</update_rate>
+    <visualize>true</visualize>
+    <topic>feeding_robot/ultrasonic/scan</topic>
+    <lidar>
+      <scan>
+        <horizontal>
+          <samples>5</samples>
+          <resolution>1</resolution>
+          <min_angle>-0.1309</min_angle>
+          <max_angle>0.1309</max_angle>
+        </horizontal>
+      </scan>
+      <range>
+        <min>0.02</min>
+        <max>4.0</max>
+        <resolution>0.01</resolution>
+      </range>
+    </lidar>
+  </sensor>
+</gazebo>
+<!-- ==================== FORCE/TORQUE SENSOR ==================== -->
+<!-- Contact/force sensor on the feeder head (spoon) joint -->
+<gazebo reference="joint4">
+  <sensor type="force_torque" name="spoon_force_sensor">
+    <always_on>true</always_on>
+    <update_rate>50.0</update_rate>
+    <visualize>true</visualize>
+    <topic>spoon/wrench</topic>
+    <force_torque>
+      <frame>child</frame>
+      <measure_direction>child_to_parent</measure_direction>
+    </force_torque>
   </sensor>
 </gazebo>

Commit message: updates

File: ros2_feedbot_ws/src/feedbot_description/urdf/my_robot.urdf.xacro (robot description, xacro)
@@ -393,10 +393,10 @@
   <parent link="feeder_head"/>
   <child link="ultrasonic_link"/>
-  <origin xyz="0.02 0 -0.015" rpy="0 0 0"/>
+  <origin xyz="0.02 0 0.02" rpy="0 0 0"/>
 </joint>
 <link name="ultrasonic_link">
   <visual>
     <geometry>
-      <box size="0.01 0.005 0.004"/>
+      <box size="0.01 0.02 0.008"/>
     </geometry>
     <material name="blue">

Commit message: updates

File: ros2_feedbot_ws/src/feedbot_description/urdf/my_robot.urdf.xacro (robot description, xacro)
@@ -222,4 +222,7 @@
           scale="0.01 0.01 0.01"/>
   </geometry>
+  <material name="apple_red">
+    <color rgba="0.9 0.1 0.05 1.0"/>
+  </material>
 </visual>
   <collision>
@@ -237,5 +240,11 @@
   </link>
 <gazebo reference="apple_link">
-  <material>Gazebo/Red</material>
+  <visual>
+    <material>
+      <ambient>0.9 0.1 0.05 1</ambient>
+      <diffuse>0.9 0.1 0.05 1</diffuse>
+      <specular>0.3 0.3 0.3 1</specular>
+    </material>
+  </visual>
 </gazebo>
 <joint name="apple_to_plate" type="fixed">
@@ -250,4 +259,7 @@
           scale="0.01 0.01 0.01"/>
   </geometry>
+  <material name="strawberry_red">
+    <color rgba="0.8 0.05 0.1 1.0"/>
+  </material>
 </visual>
   <collision>
@@ -265,5 +277,11 @@
    </link>
 <gazebo reference="strawberry_link">
-  <material>Gazebo/Red</material>
+  <visual>
+    <material>
+      <ambient>0.8 0.05 0.1 1</ambient>
+      <diffuse>0.8 0.05 0.1 1</diffuse>
+      <specular>0.2 0.2 0.2 1</specular>
+    </material>
+  </visual>
 </gazebo>
 <joint name="strawberry_to_plate" type="fixed">

Commit message: updates

File: ros2_feedbot_ws/src/feedbot_description/urdf/my_robot.urdf.xacro (robot description, xacro)
@@ -206,8 +206,20 @@
 </gazebo>
 <gazebo reference="table_link">
-  <material>Gazebo/Wood</material>
+  <visual>
+    <material>
+      <ambient>0.6 0.4 0.2 1</ambient>
+      <diffuse>0.6 0.4 0.2 1</diffuse>
+      <specular>0.1 0.1 0.1 1</specular>
+    </material>
+  </visual>
 </gazebo>
 <gazebo reference="plate_link">
-  <material>Gazebo/White</material>
+  <visual>
+    <material>
+      <ambient>0.95 0.95 0.95 1</ambient>
+      <diffuse>0.95 0.95 0.95 1</diffuse>
+      <specular>0.5 0.5 0.5 1</specular>
+    </material>
+  </visual>
 </gazebo>
 <joint name="plate_to_table" type="fixed">
@@ -289,4 +301,76 @@
   <child link="strawberry_link"/>
   <origin xyz="-0.03 0.02 0.0010"/>
+</joint>
+<!-- BANANA -->
+<link name="banana_link">
+  <visual>
+    <geometry>
+      <cylinder radius="0.012" length="0.07"/>
+    </geometry>
+    <origin xyz="0 0 0" rpy="0 1.2 0"/>
+    <material name="banana_yellow">
+      <color rgba="1.0 0.9 0.1 1.0"/>
+    </material>
+  </visual>
+  <collision>
+    <geometry>
+      <cylinder radius="0.012" length="0.07"/>
+    </geometry>
+    <origin xyz="0 0 0" rpy="0 1.2 0"/>
+  </collision>
+  <inertial>
+    <mass value="0.015"/>
+    <inertia ixx="0.00001" ixy="0" ixz="0"
+             iyy="0.00001" iyz="0" izz="0.00001"/>
+  </inertial>
+</link>
+<gazebo reference="banana_link">
+  <visual>
+    <material>
+      <ambient>1.0 0.9 0.1 1</ambient>
+      <diffuse>1.0 0.9 0.1 1</diffuse>
+      <specular>0.3 0.3 0.3 1</specular>
+    </material>
+  </visual>
+</gazebo>
+<joint name="banana_to_plate" type="fixed">
+  <parent link="plate_link"/>
+  <child link="banana_link"/>
+  <origin xyz="0.02 -0.03 0.012"/>
+</joint>
+<!-- ORANGE -->
+<link name="orange_link">
+  <visual>
+    <geometry>
+      <sphere radius="0.018"/>
+    </geometry>
+    <material name="orange_color">
+      <color rgba="1.0 0.55 0.0 1.0"/>
+    </material>
+  </visual>
+  <collision>
+    <geometry>
+      <sphere radius="0.018"/>
+    </geometry>
+  </collision>
+  <inertial>
+    <mass value="0.02"/>
+    <inertia ixx="0.00001" ixy="0" ixz="0"
+             iyy="0.00001" iyz="0" izz="0.00001"/>
+  </inertial>
+</link>
+<gazebo reference="orange_link">
+  <visual>
+    <material>
+      <ambient>1.0 0.55 0.0 1</ambient>
+      <diffuse>1.0 0.55 0.0 1</diffuse>
+      <specular>0.3 0.3 0.3 1</specular>
+    </material>
+  </visual>
+</gazebo>
+<joint name="orange_to_plate" type="fixed">
+  <parent link="plate_link"/>
+  <child link="orange_link"/>
+  <origin xyz="-0.02 -0.02 0.018"/>
 </joint>
 <!-- MOUTH OPEN MODEL (only one copy!) -->

Commit message: controller_error

File: ros2_feedbot_ws/src/feedbot_description/urdf/my_robot.urdf.xacro (robot description, xacro)
@@ -550,34 +550,30 @@
 <ros2_control name="FeedbotSystem" type="system">
   <hardware>
-    <plugin>ign_ros2_control/IgnitionSystem</plugin>
+    <plugin>gz_ros2_control/GazeboSimSystem</plugin>
   </hardware>
-<joint name="joint1">
-  <command_interface name="effort"/>
-  <state_interface name="position"/>
-  <state_interface name="velocity"/>
-  <state_interface name="effort"/>
-</joint>
-<joint name="joint2">
-  <command_interface name="effort"/>
-  <state_interface name="position"/>
-  <state_interface name="velocity"/>
-  <state_interface name="effort"/>
-</joint>
-<joint name="joint3">
-  <command_interface name="effort"/>
-  <state_interface name="position"/>
-  <state_interface name="velocity"/>
-  <state_interface name="effort"/>
-</joint>
-<joint name="joint4">
-  <command_interface name="effort"/>
-  <state_interface name="position"/>
-  <state_interface name="velocity"/>
-  <state_interface name="effort"/>
-</joint>
+  <joint name="joint1">
+    <command_interface name="position"/>
+    <state_interface name="position"/>
+    <state_interface name="velocity"/>
+  </joint>
+  <joint name="joint2">
+    <command_interface name="position"/>
+    <state_interface name="position"/>
+    <state_interface name="velocity"/>
+  </joint>
+  <joint name="joint3">
+    <command_interface name="position"/>
+    <state_interface name="position"/>
+    <state_interface name="velocity"/>
+  </joint>
+  <joint name="joint4">
+    <command_interface name="position"/>
+    <state_interface name="position"/>
+    <state_interface name="velocity"/>
+  </joint>
 </ros2_control>
 <gazebo>
-  <plugin name="ign_ros2_control::IgnitionROS2ControlPlugin"
-          filename="libign_ros2_control-system.so">
+  <plugin filename="gz_ros2_control-system"
+          name="gz_ros2_control::GazeboSimROS2ControlPlugin">
     <parameters>$(find feedbot_description)/config/controllers.yaml</parameters>
   </plugin>

Commit message: moveit2

File: ros2_feedbot_ws/src/feedbot_description/urdf/my_robot.urdf.xacro (robot description, xacro)
@@ -229,32 +229,31 @@
 </joint>
 <link name="apple_link">
-<visual>
-  <geometry>
-    <mesh filename="package://feedbot_description/meshes/apple.stl"
-          scale="0.01 0.01 0.01"/>
-  </geometry>
-  <material name="apple_red">
-    <color rgba="0.9 0.1 0.05 1.0"/>
-  </material>
-</visual>
-  <collision>
+  <visual>
     <geometry>
       <mesh filename="package://feedbot_description/meshes/apple.stl"
-            scale="0.01 0.01 0.01"/>
-    </geometry>
-  </collision>
-  <inertial>
-    <mass value="0.02"/>
-    <inertia ixx="0.00001" ixy="0" ixz="0"
-             iyy="0.00001" iyz="0"
-             izz="0.00001"/>
-  </inertial>
-  </link>
+            scale="0.025 0.025 0.025"/>
+    </geometry>
+    <material name="apple_red">
+      <color rgba="0.8 0.12 0.08 1.0"/>
+    </material>
+  </visual>
+  <collision>
+    <geometry>
+      <mesh filename="package://feedbot_description/meshes/apple.stl"
+            scale="0.025 0.025 0.025"/>
+    </geometry>
+  </collision>
+  <inertial>
+    <mass value="0.05"/>
+    <inertia ixx="0.00005" ixy="0" ixz="0"
+             iyy="0.00005" iyz="0" izz="0.00005"/>
+  </inertial>
+</link>
 <gazebo reference="apple_link">
   <visual>
     <material>
-      <ambient>0.9 0.1 0.05 1</ambient>
-      <diffuse>0.9 0.1 0.05 1</diffuse>
-      <specular>0.3 0.3 0.3 1</specular>
+      <ambient>0.7 0.05 0.02 1</ambient>
+      <diffuse>0.8 0.12 0.08 1</diffuse>
+      <specular>0.4 0.3 0.3 1</specular>
     </material>
   </visual>
@@ -263,35 +262,34 @@
   <parent link="plate_link"/>
   <child link="apple_link"/>
-  <origin xyz="0.05 0 0.0010"/>
+  <origin xyz="0.02 0.02 0.005"/>
 </joint>
 <link name="strawberry_link">
-<visual>
-  <geometry>
-    <mesh filename="package://feedbot_description/meshes/strawberry.stl"
-          scale="0.01 0.01 0.01"/>
-  </geometry>
-  <material name="strawberry_red">
-    <color rgba="0.8 0.05 0.1 1.0"/>
-  </material>
-</visual>
-  <collision>
+  <visual>
     <geometry>
       <mesh filename="package://feedbot_description/meshes/strawberry.stl"
-            scale="0.01 0.01 0.01"/>
-    </geometry>
-  </collision>
-  <inertial>
-    <mass value="0.015"/>
-    <inertia ixx="0.00001" ixy="0" ixz="0"
-             iyy="0.00001" iyz="0"
-             izz="0.00001"/>
-  </inertial>
-   </link>
+            scale="0.025 0.025 0.025"/>
+    </geometry>
+    <material name="strawberry_red">
+      <color rgba="0.85 0.15 0.18 1.0"/>
+    </material>
+  </visual>
+  <collision>
+    <geometry>
+      <mesh filename="package://feedbot_description/meshes/strawberry.stl"
+            scale="0.025 0.025 0.025"/>
+    </geometry>
+  </collision>
+  <inertial>
+    <mass value="0.03"/>
+    <inertia ixx="0.00003" ixy="0" ixz="0"
+             iyy="0.00003" iyz="0" izz="0.00003"/>
+  </inertial>
+</link>
 <gazebo reference="strawberry_link">
   <visual>
     <material>
-      <ambient>0.8 0.05 0.1 1</ambient>
-      <diffuse>0.8 0.05 0.1 1</diffuse>
-      <specular>0.2 0.2 0.2 1</specular>
+      <ambient>0.75 0.08 0.1 1</ambient>
+      <diffuse>0.85 0.15 0.18 1</diffuse>
+      <specular>0.3 0.2 0.2 1</specular>
     </material>
   </visual>
@@ -300,27 +298,27 @@
   <parent link="plate_link"/>
   <child link="strawberry_link"/>
-  <origin xyz="-0.03 0.02 0.0010"/>
-</joint>
-<!-- BANANA -->
+  <origin xyz="-0.02 -0.02 0.005"/>
+</joint>
+<!-- BANANA — realistic yellow, curved shape approximated with tilted capsule -->
 <link name="banana_link">
   <visual>
     <geometry>
-      <cylinder radius="0.012" length="0.07"/>
-    </geometry>
-    <origin xyz="0 0 0" rpy="0 1.2 0"/>
+      <cylinder radius="0.02" length="0.12"/>
+    </geometry>
+    <origin xyz="0 0 0" rpy="0 1.1 0.3"/>
     <material name="banana_yellow">
-      <color rgba="1.0 0.9 0.1 1.0"/>
-    </material>
-  </visual>
-  <collision>
-    <geometry>
-      <cylinder radius="0.012" length="0.07"/>
-    </geometry>
-    <origin xyz="0 0 0" rpy="0 1.2 0"/>
-  </collision>
-  <inertial>
-    <mass value="0.015"/>
-    <inertia ixx="0.00001" ixy="0" ixz="0"
-             iyy="0.00001" iyz="0" izz="0.00001"/>
+      <color rgba="0.95 0.85 0.15 1.0"/>
+    </material>
+  </visual>
+  <collision>
+    <geometry>
+      <cylinder radius="0.02" length="0.12"/>
+    </geometry>
+    <origin xyz="0 0 0" rpy="0 1.1 0.3"/>
+  </collision>
+  <inertial>
+    <mass value="0.04"/>
+    <inertia ixx="0.00005" ixy="0" ixz="0"
+             iyy="0.00005" iyz="0" izz="0.00005"/>
   </inertial>
 </link>
@@ -328,7 +326,7 @@
   <visual>
     <material>
-      <ambient>1.0 0.9 0.1 1</ambient>
-      <diffuse>1.0 0.9 0.1 1</diffuse>
-      <specular>0.3 0.3 0.3 1</specular>
+      <ambient>0.85 0.75 0.05 1</ambient>
+      <diffuse>0.95 0.85 0.15 1</diffuse>
+      <specular>0.2 0.2 0.1 1</specular>
     </material>
   </visual>
@@ -337,25 +335,25 @@
   <parent link="plate_link"/>
   <child link="banana_link"/>
-  <origin xyz="0.02 -0.03 0.012"/>
-</joint>
-<!-- ORANGE -->
+  <origin xyz="0.03 0.0 0.015"/>
+</joint>
+<!-- ORANGE — realistic orange sphere -->
 <link name="orange_link">
   <visual>
     <geometry>
-      <sphere radius="0.018"/>
+      <sphere radius="0.035"/>
     </geometry>
     <material name="orange_color">
-      <color rgba="1.0 0.55 0.0 1.0"/>
-    </material>
-  </visual>
-  <collision>
-    <geometry>
-      <sphere radius="0.018"/>
-    </geometry>
-  </collision>
-  <inertial>
-    <mass value="0.02"/>
-    <inertia ixx="0.00001" ixy="0" ixz="0"
-             iyy="0.00001" iyz="0" izz="0.00001"/>
+      <color rgba="1.0 0.5 0.0 1.0"/>
+    </material>
+  </visual>
+  <collision>
+    <geometry>
+      <sphere radius="0.035"/>
+    </geometry>
+  </collision>
+  <inertial>
+    <mass value="0.06"/>
+    <inertia ixx="0.00006" ixy="0" ixz="0"
+             iyy="0.00006" iyz="0" izz="0.00006"/>
   </inertial>
 </link>
@@ -363,7 +361,7 @@
   <visual>
     <material>
-      <ambient>1.0 0.55 0.0 1</ambient>
-      <diffuse>1.0 0.55 0.0 1</diffuse>
-      <specular>0.3 0.3 0.3 1</specular>
+      <ambient>0.9 0.4 0.0 1</ambient>
+      <diffuse>1.0 0.5 0.0 1</diffuse>
+      <specular>0.3 0.2 0.1 1</specular>
     </material>
   </visual>
@@ -372,5 +370,5 @@
   <parent link="plate_link"/>
   <child link="orange_link"/>
-  <origin xyz="-0.02 -0.02 0.018"/>
+  <origin xyz="-0.025 0.0 0.035"/>
 </joint>
 <!-- MOUTH OPEN MODEL (only one copy!) -->
