Commit message: update

File: ros2_feedbot_ws/src/feeding_robot/description/feeding_robot_core.xacro (robot description, xacro)
@@ -53,6 +53,6 @@
           <mesh filename="${mesh_vis}/base_link.stl" scale="${stl_scale}"/>
         </geometry>
-        <!-- CAD origin is at world origin, no offset needed -->
         <origin xyz="0 0 0" rpy="0 0 0"/>
+        <material name="dark_grey"/>
       </visual>
       <collision>
@@ -105,6 +105,6 @@
           <mesh filename="${mesh_vis}/shoulder_link.stl" scale="${stl_scale}"/>
         </geometry>
-        <!-- Offset: shift mesh so joint position (CAD X=-25,Y=0,Z=88) is at link origin -->
         <origin xyz="0.025 0 -0.088" rpy="0 0 0"/>
+        <material name="dark_grey"/>
       </visual>
       <collision>
@@ -157,6 +157,6 @@
           <mesh filename="${mesh_vis}/lower_arm_link.stl" scale="${stl_scale}"/>
         </geometry>
-        <!-- Offset: shift mesh so joint position (CAD X=-16,Y=0,Z=131) is at link origin -->
         <origin xyz="0.016 0 -0.131" rpy="0 0 0"/>
+        <material name="light_grey"/>
       </visual>
       <collision>
@@ -216,6 +216,6 @@
           <mesh filename="${mesh_vis}/upper_arm_link.stl" scale="${stl_scale}"/>
         </geometry>
-        <!-- Offset: shift mesh so elbow joint (CAD X=-5,Y=0,Z=331) is at link origin -->
         <origin xyz="0.005 0 -0.331" rpy="0 0 0"/>
+        <material name="light_grey"/>
       </visual>
       <collision>
@@ -261,5 +261,5 @@
     <child link="feeder_link"/>
     <origin xyz="${upper_arm_length} 0 0" rpy="0 0 0"/>
-    <axis xyz="0 1 0"/>
+    <axis xyz="0 -1 0"/>
     <limit lower="${-90.0 * pi / 180.0}" upper="${115.0 * pi / 180.0}"
            velocity="${max_velocity}" effort="${max_effort}"/>

File: ros2_feedbot_ws/src/feeding_robot/description/feeding_robot_ros2_control.xacro (robot description, xacro)
@@ -74,9 +74,9 @@
       <state_interface name="Torque Enable"/>
       <state_interface name="Present Input Voltage"/>
-      <param name="Position P Gain">800</param>
-      <param name="Position I Gain">100</param>
-      <param name="Position D Gain">100</param>
-      <param name="Profile Velocity">100</param>
-      <param name="Profile Acceleration">25</param>
+      <param name="Position P Gain">400</param>
+      <param name="Position I Gain">20</param>
+      <param name="Position D Gain">150</param>
+      <param name="Profile Velocity">60</param>
+      <param name="Profile Acceleration">15</param>
       <param name="Drive Mode">0</param>
       <param name="Return Delay Time">0</param>
@@ -91,9 +91,9 @@
       <state_interface name="Torque Enable"/>
       <state_interface name="Present Input Voltage"/>
-      <param name="Position P Gain">800</param>
-      <param name="Position I Gain">100</param>
-      <param name="Position D Gain">100</param>
-      <param name="Profile Velocity">100</param>
-      <param name="Profile Acceleration">25</param>
+      <param name="Position P Gain">400</param>
+      <param name="Position I Gain">20</param>
+      <param name="Position D Gain">150</param>
+      <param name="Profile Velocity">60</param>
+      <param name="Profile Acceleration">15</param>
       <param name="Drive Mode">0</param>
       <param name="Return Delay Time">0</param>
@@ -108,9 +108,9 @@
       <state_interface name="Torque Enable"/>
       <state_interface name="Present Input Voltage"/>
-      <param name="Position P Gain">800</param>
-      <param name="Position I Gain">100</param>
-      <param name="Position D Gain">100</param>
-      <param name="Profile Velocity">100</param>
-      <param name="Profile Acceleration">25</param>
+      <param name="Position P Gain">400</param>
+      <param name="Position I Gain">20</param>
+      <param name="Position D Gain">150</param>
+      <param name="Profile Velocity">60</param>
+      <param name="Profile Acceleration">15</param>
       <param name="Drive Mode">0</param>
       <param name="Return Delay Time">0</param>
@@ -125,9 +125,9 @@
       <state_interface name="Torque Enable"/>
       <state_interface name="Present Input Voltage"/>
-      <param name="Position P Gain">800</param>
-      <param name="Position I Gain">100</param>
-      <param name="Position D Gain">100</param>
-      <param name="Profile Velocity">100</param>
-      <param name="Profile Acceleration">25</param>
+      <param name="Position P Gain">400</param>
+      <param name="Position I Gain">20</param>
+      <param name="Position D Gain">150</param>
+      <param name="Profile Velocity">60</param>
+      <param name="Profile Acceleration">15</param>
       <param name="Drive Mode">0</param>
       <param name="Return Delay Time">0</param>

Commit message: update

File: ros2_feedbot_ws/src/feeding_robot/description/feeding_robot_core.xacro (robot description, xacro)
@@ -54,5 +54,4 @@
         </geometry>
         <origin xyz="0 0 0" rpy="0 0 0"/>
-        <material name="dark_grey"/>
       </visual>
       <collision>
@@ -106,5 +105,4 @@
         </geometry>
         <origin xyz="0.025 0 -0.088" rpy="0 0 0"/>
-        <material name="dark_grey"/>
       </visual>
       <collision>
@@ -158,5 +156,4 @@
         </geometry>
         <origin xyz="0.016 0 -0.131" rpy="0 0 0"/>
-        <material name="light_grey"/>
       </visual>
       <collision>
@@ -217,5 +214,4 @@
         </geometry>
         <origin xyz="0.005 0 -0.331" rpy="0 0 0"/>
-        <material name="light_grey"/>
       </visual>
       <collision>
@@ -261,5 +257,5 @@
     <child link="feeder_link"/>
     <origin xyz="${upper_arm_length} 0 0" rpy="0 0 0"/>
-    <axis xyz="0 -1 0"/>
+    <axis xyz="0 1 0"/>
     <limit lower="${-90.0 * pi / 180.0}" upper="${115.0 * pi / 180.0}"
            velocity="${max_velocity}" effort="${max_effort}"/>
@@ -411,3 +407,28 @@
     <origin xyz="${feeder_length} 0 0" rpy="0 0 0"/>
   </joint>
+  <!-- ==================== PLATE (fixed in front of robot) ==================== -->
+  <link name="plate_link">
+    <visual>
+      <geometry>
+        <mesh filename="${mesh_vis}/plate_printing.stl"/>
+      </geometry>
+      <origin xyz="0 0 0" rpy="0 0 0"/>
+    </visual>
+    <collision>
+      <geometry>
+        <mesh filename="${mesh_vis}/plate_printing.stl"/>
+      </geometry>
+    </collision>
+    <inertial>
+      <mass value="0.2"/>
+      <inertia ixx="0.001" ixy="0.0" ixz="0.0"
+               iyy="0.001" iyz="0.0" izz="0.001"/>
+    </inertial>
+  </link>
+  <joint name="plate_joint" type="fixed">
+    <parent link="world"/>
+    <child link="plate_link"/>
+    <!-- Plate position: ~15cm in front of base, at table height (below base) -->
+    <origin xyz="0.15 0.0 -0.02" rpy="0 0 0"/>
+  </joint>
 </robot>

Commit message: update

File: ros2_feedbot_ws/src/feeding_robot/description/feeding_robot_core.xacro (robot description, xacro)
@@ -140,5 +140,6 @@
     <parent link="shoulder_link"/>
     <child link="lower_arm_link"/>
-    <origin xyz="0 0 ${shoulder_joint_z - base_top_z}" rpy="0 0 0"/>
+    <!-- Offset: servo zero = arm tilted ~45° forward from vertical -->
+    <origin xyz="0 0 ${shoulder_joint_z - base_top_z}" rpy="0 0.785 0"/>
     <axis xyz="0 1 0"/>
     <limit lower="${-90.0 * pi / 180.0}" upper="${90.0 * pi / 180.0}"
@@ -198,5 +199,6 @@
     <parent link="lower_arm_link"/>
     <child link="upper_arm_link"/>
-    <origin xyz="0 0 ${lower_arm_length}" rpy="0 0 0"/>
+    <!-- Offset: servo zero = elbow bent ~-45° (horizontal arm angles down) -->
+    <origin xyz="0 0 ${lower_arm_length}" rpy="0 -0.785 0"/>
     <axis xyz="0 1 0"/>
     <limit lower="${-120.0 * pi / 180.0}" upper="${75.0 * pi / 180.0}"
@@ -429,6 +431,6 @@
     <parent link="world"/>
     <child link="plate_link"/>
-    <!-- Plate position: ~15cm in front of base, at table height (below base) -->
-    <origin xyz="0.15 0.0 -0.02" rpy="0 0 0"/>
+    <!-- Plate position: 25cm from base front (~30cm from base axis) -->
+    <origin xyz="0.30 0.0 -0.02" rpy="0 0 0"/>
   </joint>
 </robot>

Commit message: update

File: ros2_feedbot_ws/src/feeding_robot/description/feeding_robot_core.xacro (robot description, xacro)
@@ -141,5 +141,5 @@
     <child link="lower_arm_link"/>
     <!-- Offset: servo zero = arm tilted ~45° forward from vertical -->
-    <origin xyz="0 0 ${shoulder_joint_z - base_top_z}" rpy="0 0.785 0"/>
+    <origin xyz="0 0 ${shoulder_joint_z - base_top_z}" rpy="0 -0.785 0"/>
     <axis xyz="0 1 0"/>
     <limit lower="${-90.0 * pi / 180.0}" upper="${90.0 * pi / 180.0}"
@@ -199,6 +199,6 @@
     <parent link="lower_arm_link"/>
     <child link="upper_arm_link"/>
-    <!-- Offset: servo zero = elbow bent ~-45° (horizontal arm angles down) -->
-    <origin xyz="0 0 ${lower_arm_length}" rpy="0 -0.785 0"/>
+    <!-- Offset: servo zero = elbow bent ~45° forward -->
+    <origin xyz="0 0 ${lower_arm_length}" rpy="0 0.785 0"/>
     <axis xyz="0 1 0"/>
     <limit lower="${-120.0 * pi / 180.0}" upper="${75.0 * pi / 180.0}"

Commit message: update

File: ros2_feedbot_ws/src/feeding_robot/description/feeding_robot_core.xacro (robot description, xacro)
@@ -140,6 +140,5 @@
     <parent link="shoulder_link"/>
     <child link="lower_arm_link"/>
-    <!-- Offset: servo zero = arm tilted ~45° forward from vertical -->
-    <origin xyz="0 0 ${shoulder_joint_z - base_top_z}" rpy="0 -0.785 0"/>
+    <origin xyz="0 0 ${shoulder_joint_z - base_top_z}" rpy="0 0 0"/>
     <axis xyz="0 1 0"/>
     <limit lower="${-90.0 * pi / 180.0}" upper="${90.0 * pi / 180.0}"
@@ -199,6 +198,5 @@
     <parent link="lower_arm_link"/>
     <child link="upper_arm_link"/>
-    <!-- Offset: servo zero = elbow bent ~45° forward -->
-    <origin xyz="0 0 ${lower_arm_length}" rpy="0 0.785 0"/>
+    <origin xyz="0 0 ${lower_arm_length}" rpy="0 0 0"/>
     <axis xyz="0 1 0"/>
     <limit lower="${-120.0 * pi / 180.0}" upper="${75.0 * pi / 180.0}"

Commit message: update

File: ros2_feedbot_ws/src/feeding_robot/description/feeding_robot_core.xacro (robot description, xacro)
@@ -199,5 +199,5 @@
     <child link="upper_arm_link"/>
     <origin xyz="0 0 ${lower_arm_length}" rpy="0 0 0"/>
-    <axis xyz="0 1 0"/>
+    <axis xyz="0 -1 0"/>
     <limit lower="${-120.0 * pi / 180.0}" upper="${75.0 * pi / 180.0}"
            velocity="${max_velocity}" effort="${max_effort}"/>
@@ -257,5 +257,5 @@
     <child link="feeder_link"/>
     <origin xyz="${upper_arm_length} 0 0" rpy="0 0 0"/>
-    <axis xyz="0 1 0"/>
+    <axis xyz="0 -1 0"/>
     <limit lower="${-90.0 * pi / 180.0}" upper="${115.0 * pi / 180.0}"
            velocity="${max_velocity}" effort="${max_effort}"/>

Commit message: update

File: ros2_feedbot_ws/src/feeding_robot/description/feeding_robot_core.xacro (robot description, xacro)
@@ -321,5 +321,6 @@
     <parent link="feeder_link"/>
     <child link="spoon_tip_frame"/>
-    <origin xyz="${feeder_length + 0.02} 0 0" rpy="0 0 0"/>
+    <!-- Fork tip: 10cm forward of camera, 3.2cm below camera -->
+    <origin xyz="0.15 0 -0.0" rpy="0 0 0"/>
   </joint>
   <!-- ==================== CAMERA (Raspberry Pi Camera V2.1) ==================== -->
@@ -347,5 +348,6 @@
     <parent link="feeder_link"/>
     <child link="camera_link"/>
-    <origin xyz="0.03 0 0.05" rpy="0 0 0"/>
+    <!-- Camera on feeder body: fork is 10cm forward and 3.2cm below camera -->
+    <origin xyz="0.05 0 0.032" rpy="0 0 0"/>
   </joint>
   <link name="camera_optical_frame"/>
@@ -379,5 +381,6 @@
     <parent link="feeder_link"/>
     <child link="ultrasonic_link"/>
-    <origin xyz="0.03 0 -0.04" rpy="0 0 0"/>
+    <!-- Sonar: 8.9cm behind fork tip = ~6.1cm forward of feeder joint, below camera -->
+    <origin xyz="0.061 0 -0.01" rpy="0 0 0"/>
   </joint>
   <!-- ==================== LOAD CELL (HX711) ==================== -->

Commit message: update

File: ros2_feedbot_ws/src/feeding_robot/description/feeding_robot_core.xacro (robot description, xacro)
@@ -141,5 +141,5 @@
     <child link="lower_arm_link"/>
     <origin xyz="0 0 ${shoulder_joint_z - base_top_z}" rpy="0 0 0"/>
-    <axis xyz="0 1 0"/>
+    <axis xyz="0 -1 0"/>
     <limit lower="${-90.0 * pi / 180.0}" upper="${90.0 * pi / 180.0}"
            velocity="${max_velocity}" effort="${max_effort}"/>

Commit message: update

File: ros2_feedbot_ws/src/feeding_robot/description/feeding_robot_core.xacro (robot description, xacro)
@@ -54,4 +54,5 @@
         </geometry>
         <origin xyz="0 0 0" rpy="0 0 0"/>
+        <material name="dark_grey"/>
       </visual>
       <collision>
@@ -105,4 +106,5 @@
         </geometry>
         <origin xyz="0.025 0 -0.088" rpy="0 0 0"/>
+        <material name="dark_grey"/>
       </visual>
       <collision>
@@ -156,4 +158,5 @@
         </geometry>
         <origin xyz="0.016 0 -0.131" rpy="0 0 0"/>
+        <material name="light_grey"/>
       </visual>
       <collision>
@@ -214,4 +217,5 @@
         </geometry>
         <origin xyz="0.005 0 -0.331" rpy="0 0 0"/>
+        <material name="light_grey"/>
       </visual>
       <collision>
@@ -272,4 +276,5 @@
         <!-- Offset: shift mesh so wrist joint (CAD X=194,Y=0,Z=351) is at link origin -->
         <origin xyz="-0.194 0 -0.351" rpy="0 0 0"/>
+        <material name="black"/>
       </visual>
       <collision>

Commit message: update

File: ros2_feedbot_ws/src/feeding_robot/description/feeding_robot_core.xacro (robot description, xacro)
@@ -143,5 +143,5 @@
     <child link="lower_arm_link"/>
     <origin xyz="0 0 ${shoulder_joint_z - base_top_z}" rpy="0 0 0"/>
-    <axis xyz="0 -1 0"/>
+    <axis xyz="0 1 0"/>
     <limit lower="${-90.0 * pi / 180.0}" upper="${90.0 * pi / 180.0}"
            velocity="${max_velocity}" effort="${max_effort}"/>

Commit message: update

File: ros2_feedbot_ws/src/feeding_robot/description/feeding_robot_core.xacro (robot description, xacro)
@@ -326,6 +326,5 @@
     <parent link="feeder_link"/>
     <child link="spoon_tip_frame"/>
-    <!-- Fork tip: 10cm forward of camera, 3.2cm below camera -->
-    <origin xyz="0.15 0 -0.0" rpy="0 0 0"/>
+    <origin xyz="${feeder_length + 0.02} 0 0" rpy="0 0 0"/>
   </joint>
   <!-- ==================== CAMERA (Raspberry Pi Camera V2.1) ==================== -->
@@ -353,6 +352,5 @@
     <parent link="feeder_link"/>
     <child link="camera_link"/>
-    <!-- Camera on feeder body: fork is 10cm forward and 3.2cm below camera -->
-    <origin xyz="0.05 0 0.032" rpy="0 0 0"/>
+    <origin xyz="0.03 0 0.05" rpy="0 0 0"/>
   </joint>
   <link name="camera_optical_frame"/>
@@ -386,6 +384,5 @@
     <parent link="feeder_link"/>
     <child link="ultrasonic_link"/>
-    <!-- Sonar: 8.9cm behind fork tip = ~6.1cm forward of feeder joint, below camera -->
-    <origin xyz="0.061 0 -0.01" rpy="0 0 0"/>
+    <origin xyz="0.03 0 -0.04" rpy="0 0 0"/>
   </joint>
   <!-- ==================== LOAD CELL (HX711) ==================== -->

Commit message: update

File: ros2_feedbot_ws/src/feeding_robot/description/feeding_robot_core.xacro (robot description, xacro)
@@ -332,14 +332,12 @@
     <visual>
       <geometry>
-        <mesh filename="${mesh_vis}/camera.stl" scale="${stl_scale}"/>
-      </geometry>
-      <!-- CAD origin offset minus camera_joint offset (0.03, 0, 0.05) -->
-      <origin xyz="${-0.194 - 0.03} 0 ${-0.351 - 0.05}" rpy="0 0 0"/>
+        <box size="0.025 0.024 0.009"/>
+      </geometry>
+      <material name="green"/>
     </visual>
     <collision>
       <geometry>
-        <mesh filename="${mesh_vis}/camera.stl" scale="${stl_scale}"/>
-      </geometry>
-      <origin xyz="${-0.194 - 0.03} 0 ${-0.351 - 0.05}" rpy="0 0 0"/>
+        <box size="0.025 0.024 0.009"/>
+      </geometry>
     </collision>
     <inertial>
@@ -364,14 +362,12 @@
     <visual>
       <geometry>
-        <mesh filename="${mesh_vis}/sonar.stl" scale="${stl_scale}"/>
-      </geometry>
-      <!-- CAD origin offset minus ultrasonic_joint offset; Y shifted from CAD side (116mm) to face -->
-      <origin xyz="${-0.194 - 0.03} -0.116 ${-0.351 + 0.04}" rpy="0 0 0"/>
+        <box size="0.045 0.020 0.015"/>
+      </geometry>
+      <material name="blue"/>
     </visual>
     <collision>
       <geometry>
-        <mesh filename="${mesh_vis}/sonar.stl" scale="${stl_scale}"/>
-      </geometry>
-      <origin xyz="${-0.194 - 0.03} -0.116 ${-0.351 + 0.04}" rpy="0 0 0"/>
+        <box size="0.045 0.020 0.015"/>
+      </geometry>
     </collision>
     <inertial>
@@ -434,6 +430,6 @@
     <parent link="world"/>
     <child link="plate_link"/>
-    <!-- Plate position: 25cm from base front (~30cm from base axis) -->
-    <origin xyz="0.30 0.0 -0.02" rpy="0 0 0"/>
+    <!-- Plate: 25cm from base front, on table surface below feeder head -->
+    <origin xyz="0.25 0.0 -0.10" rpy="0 0 0"/>
   </joint>
 </robot>

Commit message: update

File: ros2_feedbot_ws/src/feeding_robot/description/feeding_robot_core.xacro (robot description, xacro)
@@ -414,5 +414,5 @@
         <mesh filename="${mesh_vis}/plate_printing.stl"/>
       </geometry>
-      <origin xyz="0 0 0" rpy="0 0 0"/>
+      <origin xyz="0 0 ${base_top_z}" rpy="0 0 0"/>
     </visual>
     <collision>

Commit message: update

File: ros2_feedbot_ws/src/feeding_robot/description/feeding_robot_core.xacro (robot description, xacro)
@@ -414,5 +414,5 @@
         <mesh filename="${mesh_vis}/plate_printing.stl"/>
       </geometry>
-      <origin xyz="0 0 ${base_top_z}" rpy="0 0 0"/>
+      <origin xyz="0 0 0" rpy="0 0 0"/>
     </visual>
     <collision>
@@ -431,5 +431,5 @@
     <child link="plate_link"/>
     <!-- Plate: 25cm from base front, on table surface below feeder head -->
-    <origin xyz="0.25 0.0 -0.10" rpy="0 0 0"/>
+    <origin xyz="0.25 0.25 -0.10" rpy="0 0 0"/>
   </joint>
 </robot>

Commit message: update

File: ros2_feedbot_ws/src/feeding_robot/description/feeding_robot_core.xacro (robot description, xacro)
@@ -332,12 +332,13 @@
     <visual>
       <geometry>
-        <box size="0.025 0.024 0.009"/>
-      </geometry>
-      <material name="green"/>
+        <mesh filename="${mesh_vis}/camera.stl" scale="${stl_scale}"/>
+      </geometry>
+      <origin xyz="${-0.194 - 0.03} 0 ${-0.351 + 0.05}" rpy="0 0 0"/>
     </visual>
     <collision>
       <geometry>
-        <box size="0.025 0.024 0.009"/>
-      </geometry>
+        <mesh filename="${mesh_vis}/camera.stl" scale="${stl_scale}"/>
+      </geometry>
+      <origin xyz="${-0.194 - 0.03} 0 ${-0.351 + 0.05}" rpy="0 0 0"/>
     </collision>
     <inertial>
@@ -362,12 +363,13 @@
     <visual>
       <geometry>
-        <box size="0.045 0.020 0.015"/>
-      </geometry>
-      <material name="blue"/>
+        <mesh filename="${mesh_vis}/sonar.stl" scale="${stl_scale}"/>
+      </geometry>
+      <origin xyz="${-0.194 - 0.03} -0.116 ${-0.351 - 0.04}" rpy="0 0 0"/>
     </visual>
     <collision>
       <geometry>
-        <box size="0.045 0.020 0.015"/>
-      </geometry>
+        <mesh filename="${mesh_vis}/sonar.stl" scale="${stl_scale}"/>
+      </geometry>
+      <origin xyz="${-0.194 - 0.03} -0.116 ${-0.351 - 0.04}" rpy="0 0 0"/>
     </collision>
     <inertial>
@@ -431,5 +433,5 @@
     <child link="plate_link"/>
     <!-- Plate: 25cm from base front, on table surface below feeder head -->
-    <origin xyz="0.25 0.25 -0.10" rpy="0 0 0"/>
+    <origin xyz="-0.25 0 -0.10" rpy="0 0 0"/>
   </joint>
 </robot>

Commit message: update

File: ros2_feedbot_ws/src/feeding_robot/description/feeding_robot_core.xacro (robot description, xacro)
@@ -342,4 +342,5 @@
       <origin xyz="${-0.194 - 0.03} 0 ${-0.351 + 0.05}" rpy="0 0 0"/>
     </collision>
+    </collision>
     <inertial>
       <mass value="0.003"/>
@@ -351,5 +352,5 @@
     <parent link="feeder_link"/>
     <child link="camera_link"/>
-    <origin xyz="0.03 0 0.05" rpy="0 0 0"/>
+    <origin xyz="0.03 0 -0.05" rpy="0 0 0"/>
   </joint>
   <link name="camera_optical_frame"/>
@@ -382,5 +383,5 @@
     <parent link="feeder_link"/>
     <child link="ultrasonic_link"/>
-    <origin xyz="0.03 0 -0.04" rpy="0 0 0"/>
+    <origin xyz="0.03 0 0.04" rpy="0 0 0"/>
   </joint>
   <!-- ==================== LOAD CELL (HX711) ==================== -->
@@ -432,6 +433,6 @@
     <parent link="world"/>
     <child link="plate_link"/>
-    <!-- Plate: 25cm from base front, on table surface below feeder head -->
-    <origin xyz="-0.25 0 -0.10" rpy="0 0 0"/>
+    <!-- Plate: below feeder head (arm extends to -X in RViz due to flipped axes) -->
+    <origin xyz="-0.25 0.0 -0.15" rpy="0 0 0"/>
   </joint>
 </robot>

Commit message: update

File: ros2_feedbot_ws/src/feeding_robot/description/feeding_robot_core.xacro (robot description, xacro)
@@ -342,5 +342,4 @@
       <origin xyz="${-0.194 - 0.03} 0 ${-0.351 + 0.05}" rpy="0 0 0"/>
     </collision>
-    </collision>
     <inertial>
       <mass value="0.003"/>

Commit message: update

File: ros2_feedbot_ws/src/feeding_robot/description/feeding_robot_core.xacro (robot description, xacro)
@@ -104,5 +104,5 @@
           <mesh filename="${mesh_vis}/shoulder_link.stl" scale="${stl_scale}"/>
         </geometry>
-        <origin xyz="0.025 0 -0.088" rpy="0 0 0"/>
+        <origin xyz="0 0 -0.088" rpy="0 0 0"/>
         <material name="dark_grey"/>
       </visual>
@@ -111,5 +111,5 @@
           <mesh filename="${mesh_col}/shoulder_link.stl" scale="${stl_scale}"/>
         </geometry>
-        <origin xyz="0.025 0 -0.088" rpy="0 0 0"/>
+        <origin xyz="0 0 -0.088" rpy="0 0 0"/>
       </collision>
     </xacro:if>

Commit message: update

File: ros2_feedbot_ws/src/feeding_robot/description/feeding_robot_core.xacro (robot description, xacro)
@@ -104,4 +104,5 @@
           <mesh filename="${mesh_vis}/shoulder_link.stl" scale="${stl_scale}"/>
         </geometry>
+        <!-- Shift mesh so base_y_joint (CAD 0,0,88) is at link origin -->
         <origin xyz="0 0 -0.088" rpy="0 0 0"/>
         <material name="dark_grey"/>
@@ -141,5 +142,6 @@
     <parent link="shoulder_link"/>
     <child link="lower_arm_link"/>
-    <origin xyz="0 0 ${shoulder_joint_z - base_top_z}" rpy="0 0 0"/>
+    <!-- Shoulder joint in CAD: (-16, 0, 131) mm, relative to base top (0,0,88) -->
+    <origin xyz="-0.016 0 ${shoulder_joint_z - base_top_z}" rpy="0 0 0"/>
     <axis xyz="0 1 0"/>
     <limit lower="${-90.0 * pi / 180.0}" upper="${90.0 * pi / 180.0}"
@@ -200,5 +202,6 @@
     <parent link="lower_arm_link"/>
     <child link="upper_arm_link"/>
-    <origin xyz="0 0 ${lower_arm_length}" rpy="0 0 0"/>
+    <!-- Elbow joint in CAD: (-5, 0, 331) mm, relative to shoulder (-16, 0, 131) -->
+    <origin xyz="0.011 0 ${lower_arm_length}" rpy="0 0 0"/>
     <axis xyz="0 -1 0"/>
     <limit lower="${-120.0 * pi / 180.0}" upper="${75.0 * pi / 180.0}"
@@ -432,5 +435,6 @@
     <child link="plate_link"/>
     <!-- Plate: below feeder head (arm extends to -X in RViz due to flipped axes) -->
-    <origin xyz="-0.25 0.0 -0.15" rpy="0 0 0"/>
+    <!--origin xyz="-0.25 0.0 -0.15" rpy="0 0 0"/-->
+    <origin xyz="0.25 -0.25 0.050" rpy="0 0 0"/>
   </joint>
 </robot>
