Commit message: update

File: ros2_feedbot_ws/src/feeding_robot/description/feeding_robot_core.xacro (robot description, xacro)
@@ -142,6 +142,5 @@
     <parent link="shoulder_link"/>
     <child link="lower_arm_link"/>
-    <!-- Shoulder joint in CAD: (-16, 0, 131) mm, relative to base top (0,0,88) -->
-    <origin xyz="-0.016 0 ${shoulder_joint_z - base_top_z}" rpy="0 0 0"/>
+    <origin xyz="0 0 ${shoulder_joint_z - base_top_z}" rpy="0 0 0"/>
     <axis xyz="0 1 0"/>
     <limit lower="${-90.0 * pi / 180.0}" upper="${90.0 * pi / 180.0}"
@@ -202,6 +201,5 @@
     <parent link="lower_arm_link"/>
     <child link="upper_arm_link"/>
-    <!-- Elbow joint in CAD: (-5, 0, 331) mm, relative to shoulder (-16, 0, 131) -->
-    <origin xyz="0.011 0 ${lower_arm_length}" rpy="0 0 0"/>
+    <origin xyz="0 0 ${lower_arm_length}" rpy="0 0 0"/>
     <axis xyz="0 -1 0"/>
     <limit lower="${-120.0 * pi / 180.0}" upper="${75.0 * pi / 180.0}"
